File: NeoCoreShield2.sch (EAGLE design)
At the start: 41 parts, among them J6 BINDER_M12_PAR_8_DIP, J7 BINDER_M12_PAR_8_DIP, J8 BINDER_M12_PAR_8_DIP, J9 BINDER_M12_PAR_8_DIP, Q1 2.5A/30V/105mΩ, Q2 310mA/60V/1.6Ω, Q3 2.5A/30V/105mΩ, Q4 2.5A/30V/105mΩ, Q5 310mA/60V/1.6Ω, Q6 310mA/60V/1.6Ω

Commit message: Routed Neo Core Shields
Parts:
- added JP5, JP6, JP7, JP8: JUMPER-SMT_2_NO_SILK, SparkFun-Jumpers:JUMPER-SMT_2_NO_SILK
Connections:
- new net UART_RX_TX: J11.3, JP5.1, JP6.1
- new net UART_TX_RX: J11.4, JP7.1, JP8.1
- net GND: now also J6.BROWN, J7.BROWN, J8.BROWN; no longer J6.WHITE, J7.WHITE, J8.WHITE
- net LED_CONTROL1: now also U1G$1.MP
- net LED_CONTROL2: now also U1G$3.SCL
- net UART_RX: now also JP5.2, JP7.2; no longer J11.4
- net UART_TX: now also JP6.2, JP8.2; no longer J11.3
- net USB_CAM_1_N: now also J6.WHITE; no longer J6.BROWN
- net USB_CAM_2_N: now also J7.WHITE; no longer J7.BROWN
- net USB_CAM_3_N: now also J8.WHITE; no longer J8.BROWN
Other:
- moved on the sheet: U1G$3
